Commit message: code update

File: chapter6/chapt6_ws/install/robot_description2/share/robot_description2/urdf/robot/base.urdf.xacro (robot description, xacro)
@@ -47,4 +47,8 @@
             <child link="base_link"/>
         </joint>
+        <!-- 给 gazebo 提供的标签【颜色...】 -->
+        <gazebo reference="base_link">
+            <material>Gazebo/Grey</material>
+        </gazebo>
     </xacro:macro>
 </robot>

File: chapter6/chapt6_ws/install/robot_description2/share/robot_description2/urdf/robot/sensor/camera.urdf.xacro (robot description, xacro)
@@ -42,4 +42,8 @@
             <origin xyz="${xyz}" rpy="0.0 0.0 0.0"/>
         </joint>
+        <!-- 给 gazebo 提供的标签【颜色...】 -->
+        <gazebo reference="camera_link">
+            <material>Gazebo/Black</material>
+        </gazebo>
     </xacro:macro>
 </robot>

File: chapter6/chapt6_ws/install/robot_description2/share/robot_description2/urdf/robot/sensor/imu.urdf.xacro (robot description, xacro)
@@ -42,4 +42,8 @@
             <origin xyz="${xyz}" rpy="0.0 0.0 0.0"/>
         </joint>
+        <!-- 给 gazebo 提供的标签【颜色...】 -->
+        <gazebo reference="imu_link">
+            <material>Gazebo/Red</material>
+        </gazebo>
     </xacro:macro>
 </robot>
