Commit message: code update

File: chapter6/chapt6_ws/install/robot_description2/share/robot_description2/urdf/robot/robot.urdf.xacro (robot description, xacro)
@@ -12,4 +12,7 @@
 <xacro:include filename="$(find robot_description2)/urdf/robot/actuator/wheel.urdf.xacro"/>
 <xacro:include filename="$(find robot_description2)/urdf/robot/actuator/caster.urdf.xacro"/>
+<!-- 插件部分 -->
+<xacro:include filename="$(find robot_description2)/urdf/robot/plugins/gazebo_control_plugins.xacro"/>
+<xacro:include filename="$(find robot_description2)/urdf/robot/plugins/gazebo_sensor_plugins.xacro"/>
 <!-- 调用宏 xacro -->
 <xacro:base_xacro length="0.12" radius="0.1"/>
@@ -21,3 +24,5 @@
 <xacro:caster_xacro caster_name="front_caster" xyz="0.08 0.0 -0.076"/>
 <xacro:caster_xacro caster_name="back_caster" xyz="-0.08 0.0 -0.076"/>
+<xacro:gazebo_control_plugin/>
+<xacro:gazebo_sensor_plugin/>
 </robot>

File: chapter6/chapt6_ws/install/robot_description2/share/robot_description2/urdf/robot/sensor/camera.urdf.xacro (robot description, xacro)
@@ -4,4 +4,6 @@
     <xacro:include filename="$(find robot_description2)/urdf/robot/common_inertia.xacro"/>
     <xacro:macro name="camera_xacro" params="xyz">
+        <!-- 虚拟 link -->
+        <link name="camera_optical_link"></link>
         <!-- 机器人的 camera 部件 -->
         <link name="camera_link">
@@ -42,4 +44,12 @@
             <origin xyz="${xyz}" rpy="0.0 0.0 0.0"/>
         </joint>
+        <!-- 机器人的关节，用于组合机器人的部件 -->
+        <joint name="camera_optical_joint" type="fixed">
+            <parent link="camera_link"/>
+            <child link="camera_optical_link"/>
+            <!-- 将 camera_optical_link 固定在 camera_link 几何中心的偏移处 -->
+            <!-- 相机朝向默认前方为 z 轴，因此要进行修正，旋转 90 度 -->
+            <origin xyz="0.0 0.0 0.0" rpy="${-pi/2} 0.0 ${-pi/2}"/>
+        </joint>
         <!-- 给 gazebo 提供的标签【颜色...】 -->
         <gazebo reference="camera_link">
