Commit message: code update

File: chapter6/chapt6_ws/install/robot_description2/share/robot_description2/urdf/robot/actuator/caster.urdf.xacro (robot description, xacro)
@@ -18,4 +18,17 @@
                 </material>
             </visual>
+            <collision>
+                <!-- 沿着自己几何中心的偏移和旋转量 -->
+                <!-- 轮子要翻转 90 度 -->
+                <origin xyz="0.0 0.0 0.0" rpy="0.0 0.0 0.0"/>
+                <!-- 几何形状 -->
+                <geometry>
+                    <sphere radius="0.016"/>
+                </geometry>
+                <!-- 材质和颜色 -->
+                <material name="yellow">
+                    <color rgba="1.0 1.0 0.0 0.8"/>
+                </material>
+            </collision>
         </link>
         <!-- 机器人的关节，用于组合机器人的部件 -->

File: chapter6/chapt6_ws/install/robot_description2/share/robot_description2/urdf/robot/actuator/wheel.urdf.xacro (robot description, xacro)
@@ -18,4 +18,17 @@
                 </material>
             </visual>
+            <collision>
+                <!-- 沿着自己几何中心的偏移和旋转量 -->
+                <!-- 轮子要翻转 90 度 -->
+                <origin xyz="0.0 0.0 0.0" rpy="1.57079 0.0 0.0"/>
+                <!-- 几何形状 -->
+                <geometry>
+                    <cylinder radius="0.032" length="0.04"/>
+                </geometry>
+                <!-- 材质和颜色 -->
+                <material name="yellow">
+                    <color rgba="1.0 1.0 0.0 0.8"/>
+                </material>
+            </collision>
         </link>
         <!-- 机器人的关节，用于组合机器人的部件 -->

File: chapter6/chapt6_ws/install/robot_description2/share/robot_description2/urdf/robot/base.urdf.xacro (robot description, xacro)
@@ -2,4 +2,6 @@
 <robot xmlns:xacro="http://www.ros.org/wiki/xacro">
     <xacro:macro name="base_xacro" params="radius length">
+        <!-- 虚拟部件【有 link、joint，但是没有实体】 -->
+        <link name="base_footprint"/>
         <!-- 机器人的身体部分 -->
         <link name="base_link">
@@ -18,5 +20,28 @@
                 </material>
             </visual>
+            <!-- 添加碰撞属性[可以和 visual 标签的一样，也可以不一样] -->
+            <collision>
+                <!-- 沿着自己几何中心的偏移和旋转量 -->
+                <origin xyz="0.0 0.0 0.0" rpy="0.0 0.0 0.0"/>
+                <!-- 几何形状 -->
+                <geometry>
+                    <!-- 圆柱体：{半径：0.10米， 高度：0.12米} -->
+                    <cylinder radius="${radius}" length="${length}"/>
+                </geometry>
+                <!-- 材质和颜色 -->
+                <material name="white">
+                    <color rgba="1.0 1.0 1.0 0.5"/>
+                </material>
+            </collision>
         </link>
+        <!-- 虚拟部件【有 link、joint，但是没有实体】 -->
+        <joint name="base_footprint_joint" type="fixed">
+            <!-- base_link 在地面上的投影 -->
+            <!-- 机身的一半高度+轮子半径， “-0.001”是为了紧贴地面 -->
+            <!-- length / 2 + 0.032 - 0.001 -->
+            <origin xyz="0.0 0.0 ${length/2+0.032-0.001}" rpy="0.0 0.0 0.0"/>
+            <parent link="base_footprint"/>
+            <child link="base_link"/>
+        </joint>
     </xacro:macro>
 </robot>

File: chapter6/chapt6_ws/install/robot_description2/share/robot_description2/urdf/robot/sensor/camera.urdf.xacro (robot description, xacro)
@@ -18,4 +18,17 @@
                 </material>
             </visual>
+            <collision>
+                <!-- 沿着自己几何中心的偏移和旋转量 -->
+                <origin xyz="0.0 0.0 0.0" rpy="0.0 0.0 0.0"/>
+                <!-- 几何形状 -->
+                <geometry>
+                    <!-- 正方体：{长：， 宽：， 高：} -->
+                    <box size="0.02 0.10 0.02"/>
+                </geometry>
+                <!-- 材质和颜色 -->
+                <material name="black">
+                    <color rgba="0.0 0.0 0.0 0.5"/>
+                </material>
+            </collision>
         </link>
         <!-- 机器人的关节，用于组合机器人的部件 -->

File: chapter6/chapt6_ws/install/robot_description2/share/robot_description2/urdf/robot/sensor/imu.urdf.xacro (robot description, xacro)
@@ -18,4 +18,17 @@
                 </material>
             </visual>
+            <collision>
+                <!-- 沿着自己几何中心的偏移和旋转量 -->
+                <origin xyz="0.0 0.0 0.0" rpy="0.0 0.0 0.0"/>
+                <!-- 几何形状 -->
+                <geometry>
+                    <!-- 正方体：{长：， 宽：， 高：} -->
+                    <box size="0.02 0.02 0.02"/>
+                </geometry>
+                <!-- 材质和颜色 -->
+                <material name="black">
+                    <color rgba="0.0 0.0 0.0 0.5"/>
+                </material>
+            </collision>
         </link>
         <!-- 机器人的关节，用于组合机器人的部件 -->

File: chapter6/chapt6_ws/install/robot_description2/share/robot_description2/urdf/robot/sensor/laser.urdf.xacro (robot description, xacro)
@@ -17,4 +17,16 @@
                 </material>
             </visual>
+            <collision>
+                <!-- 沿着自己几何中心的偏移和旋转量 -->
+                <origin xyz="0.0 0.0 0.0" rpy="0.0 0.0 0.0"/>
+                <!-- 几何形状 -->
+                <geometry>
+                    <cylinder radius="0.01" length="0.10"/>
+                </geometry>
+                <!-- 材质和颜色 -->
+                <material name="black">
+                    <color rgba="0.0 0.0 0.0 1.0"/>
+                </material>
+            </collision>
         </link>
         <!-- 雷达部件 -->
@@ -33,4 +45,16 @@
                 </material>
             </visual>
+            <collision>
+                <!-- 沿着自己几何中心的偏移和旋转量 -->
+                <origin xyz="0.0 0.0 0.0" rpy="0.0 0.0 0.0"/>
+                <!-- 几何形状 -->
+                <geometry>
+                    <cylinder radius="0.02" length="0.02"/>
+                </geometry>
+                <!-- 材质和颜色 -->
+                <material name="black">
+                    <color rgba="0.0 0.0 0.0 1.0"/>
+                </material>
+            </collision>
         </link>
         <!-- 机器人的关节，用于组合机器人的部件 -->

Commit message: code update

File: chapter6/chapt6_ws/install/robot_description2/share/robot_description2/urdf/robot/actuator/caster.urdf.xacro (robot description, xacro)
@@ -42,4 +42,18 @@
             <origin xyz="${xyz}" rpy="0.0 0.0 0.0"/>
         </joint>
+        <!-- 给 gazebo 提供的标签【颜色...】 -->
+        <gazebo reference="${caster_name}_link">
+            <material>Gazebo/Green</material>
+        </gazebo>
+        <gazebo reference="${caster_name}_link">
+            <!-- 【切向】摩擦系数 -->
+            <mu1 value="0.0"/>
+            <!-- 【法向】摩擦系数 -->
+            <mu2 value="0.0"/>
+            <!-- 刚度系数 -->
+            <kp value="1000000000.0"/>
+            <!-- 阻尼系数 -->
+            <kd value="1.0"/>
+        </gazebo>
     </xacro:macro>
 </robot>

File: chapter6/chapt6_ws/install/robot_description2/share/robot_description2/urdf/robot/actuator/wheel.urdf.xacro (robot description, xacro)
@@ -44,4 +44,18 @@
             <axis xyz="0.0 1.0 0.0"/>
         </joint>
+        <!-- 给 gazebo 提供的标签【颜色...】 -->
+        <gazebo reference="${wheel_name}_link">
+            <material>Gazebo/Yellow</material>
+        </gazebo>
+        <gazebo reference="${wheel_name}_link">
+            <!-- 【切向】摩擦系数 -->
+            <mu1 value="20.0"/>
+            <!-- 【法向】摩擦系数 -->
+            <mu2 value="20.0"/>
+            <!-- 刚度系数 -->
+            <kp value="1000000000.0"/>
+            <!-- 阻尼系数 -->
+            <kd value="1.0"/>
+        </gazebo>
     </xacro:macro>
 </robot>

File: chapter6/chapt6_ws/install/robot_description2/share/robot_description2/urdf/robot/sensor/laser.urdf.xacro (robot description, xacro)
@@ -79,4 +79,11 @@
             <origin xyz="${xyz}" rpy="0.0 0.0 0.0"/>
         </joint>
+        <!-- 给 gazebo 提供的标签【颜色...】 -->
+        <gazebo reference="laser_cylinder_link">
+            <material>Gazebo/Black</material>
+        </gazebo>
+        <gazebo reference="laser_link">
+            <material>Gazebo/Black</material>
+        </gazebo>
     </xacro:macro>
 </robot>
