Commit message: code update

File: chapter6/chapt6_ws/install/robot_description2/share/robot_description2/urdf/robot/actuator/caster.urdf.xacro (robot description, xacro)
@@ -1,19 +1,12 @@
 <?xml version="1.0"?>
 <robot xmlns:xacro="http://www.ros.org/wiki/xacro">
-    <!-- 引入已经构建好的 xacro 文件 -->
     <xacro:include filename="$(find robot_description2)/urdf/robot/common_inertia.xacro"/>
     <xacro:macro name="caster_xacro" params="caster_name xyz">
-        <!-- 机器人的 caster 部件 -->
         <link name="${caster_name}_link">
-            <!-- 部件的外观描述 -->
             <visual>
-                <!-- 沿着自己几何中心的偏移和旋转量 -->
-                <!-- 轮子要翻转 90 度 -->
                 <origin xyz="0.0 0.0 0.0" rpy="0.0 0.0 0.0"/>
-                <!-- 几何形状 -->
                 <geometry>
                     <sphere radius="0.016"/>
                 </geometry>
-                <!-- 材质和颜色 -->
                 <material name="yellow">
                     <color rgba="1.0 1.0 0.0 0.8"/>
@@ -21,12 +14,8 @@
             </visual>
             <collision>
-                <!-- 沿着自己几何中心的偏移和旋转量 -->
-                <!-- 轮子要翻转 90 度 -->
                 <origin xyz="0.0 0.0 0.0" rpy="0.0 0.0 0.0"/>
-                <!-- 几何形状 -->
                 <geometry>
                     <sphere radius="0.016"/>
                 </geometry>
-                <!-- 材质和颜色 -->
                 <material name="yellow">
                     <color rgba="1.0 1.0 0.0 0.8"/>
@@ -35,5 +24,4 @@
             <xacro:sphere_inertia m="0.05" r="0.016"/>
         </link>
-        <!-- 机器人的关节，用于组合机器人的部件 -->
         <joint name="${caster_name}_joint" type="fixed">
             <parent link="base_link"/>
@@ -42,16 +30,11 @@
             <origin xyz="${xyz}" rpy="0.0 0.0 0.0"/>
         </joint>
-        <!-- 给 gazebo 提供的标签【颜色...】 -->
         <gazebo reference="${caster_name}_link">
             <material>Gazebo/Green</material>
         </gazebo>
         <gazebo reference="${caster_name}_link">
-            <!-- 【切向】摩擦系数 -->
             <mu1 value="0.0"/>
-            <!-- 【法向】摩擦系数 -->
             <mu2 value="0.0"/>
-            <!-- 刚度系数 -->
             <kp value="1000000000.0"/>
-            <!-- 阻尼系数 -->
             <kd value="1.0"/>
         </gazebo>

File: chapter6/chapt6_ws/install/robot_description2/share/robot_description2/urdf/robot/actuator/wheel.urdf.xacro (robot description, xacro)
@@ -1,19 +1,12 @@
 <?xml version="1.0"?>
 <robot xmlns:xacro="http://www.ros.org/wiki/xacro">
-    <!-- 引入已经构建好的 xacro 文件 -->
     <xacro:include filename="$(find robot_description2)/urdf/robot/common_inertia.xacro"/>
     <xacro:macro name="wheel_xacro" params="wheel_name xyz">
-        <!-- 机器人的 wheel 部件 -->
         <link name="${wheel_name}_link">
-            <!-- 部件的外观描述 -->
             <visual>
-                <!-- 沿着自己几何中心的偏移和旋转量 -->
-                <!-- 轮子要翻转 90 度 -->
                 <origin xyz="0.0 0.0 0.0" rpy="1.57079 0.0 0.0"/>
-                <!-- 几何形状 -->
                 <geometry>
                     <cylinder radius="0.032" length="0.04"/>
                 </geometry>
-                <!-- 材质和颜色 -->
                 <material name="yellow">
                     <color rgba="1.0 1.0 0.0 0.8"/>
@@ -21,12 +14,8 @@
             </visual>
             <collision>
-                <!-- 沿着自己几何中心的偏移和旋转量 -->
-                <!-- 轮子要翻转 90 度 -->
                 <origin xyz="0.0 0.0 0.0" rpy="1.57079 0.0 0.0"/>
-                <!-- 几何形状 -->
                 <geometry>
                     <cylinder radius="0.032" length="0.04"/>
                 </geometry>
-                <!-- 材质和颜色 -->
                 <material name="yellow">
                     <color rgba="1.0 1.0 0.0 0.8"/>
@@ -35,25 +24,16 @@
             <xacro:cylinder_inertia m="0.05" r="0.032" h="0.04"/>
         </link>
-        <!-- 机器人的关节，用于组合机器人的部件 -->
         <joint name="${wheel_name}_joint" type="continuous">
             <parent link="base_link"/>
             <child link="${wheel_name}_link"/>
-            <!-- 将 wheel 固定在 base_link 几何中心的偏移处 -->
             <origin xyz="${xyz}" rpy="0.0 0.0 0.0"/>
-            <!-- 设置转动轴: 绕y轴旋转 -->
-            <axis xyz="0.0 1.0 0.0"/>
         </joint>
-        <!-- 给 gazebo 提供的标签【颜色...】 -->
         <gazebo reference="${wheel_name}_link">
             <material>Gazebo/Yellow</material>
         </gazebo>
         <gazebo reference="${wheel_name}_link">
-            <!-- 【切向】摩擦系数 -->
             <mu1 value="20.0"/>
-            <!-- 【法向】摩擦系数 -->
             <mu2 value="20.0"/>
-            <!-- 刚度系数 -->
             <kp value="1000000000.0"/>
-            <!-- 阻尼系数 -->
             <kd value="1.0"/>
         </gazebo>

File: chapter6/chapt6_ws/install/robot_description2/share/robot_description2/urdf/robot/base.urdf.xacro (robot description, xacro)
@@ -1,35 +1,22 @@
 <?xml version="1.0"?>
 <robot xmlns:xacro="http://www.ros.org/wiki/xacro">
-    <!-- 引入已经构建好的 xacro 文件 -->
     <xacro:include filename="$(find robot_description2)/urdf/robot/common_inertia.xacro"/>
     <xacro:macro name="base_xacro" params="radius length">
-        <!-- 虚拟部件【有 link、joint，但是没有实体】 -->
         <link name="base_footprint"/>
-        <!-- 机器人的身体部分 -->
         <link name="base_link">
-            <!-- 部件的外观描述 -->
             <visual>
-                <!-- 沿着自己几何中心的偏移和旋转量 -->
                 <origin xyz="0.0 0.0 0.0" rpy="0.0 0.0 0.0"/>
-                <!-- 几何形状 -->
                 <geometry>
-                    <!-- 圆柱体：{半径：0.10米， 高度：0.12米} -->
                     <cylinder radius="${radius}" length="${length}"/>
                 </geometry>
-                <!-- 材质和颜色 -->
                 <material name="white">
                     <color rgba="1.0 1.0 1.0 0.5"/>
                 </material>
             </visual>
-            <!-- 添加碰撞属性[可以和 visual 标签的一样，也可以不一样] -->
             <collision>
-                <!-- 沿着自己几何中心的偏移和旋转量 -->
                 <origin xyz="0.0 0.0 0.0" rpy="0.0 0.0 0.0"/>
-                <!-- 几何形状 -->
                 <geometry>
-                    <!-- 圆柱体：{半径：0.10米， 高度：0.12米} -->
                     <cylinder radius="${radius}" length="${length}"/>
                 </geometry>
-                <!-- 材质和颜色 -->
                 <material name="white">
                     <color rgba="1.0 1.0 1.0 0.5"/>
@@ -38,14 +25,9 @@
             <xacro:cylinder_inertia m="1.0" r="${radius}" h="${length}"/>
         </link>
-        <!-- 虚拟部件【有 link、joint，但是没有实体】 -->
         <joint name="base_footprint_joint" type="fixed">
-            <!-- base_link 在地面上的投影 -->
-            <!-- 机身的一半高度+轮子半径， “-0.001”是为了紧贴地面 -->
-            <!-- length / 2 + 0.032 - 0.001 -->
             <origin xyz="0.0 0.0 ${length/2+0.032-0.001}" rpy="0.0 0.0 0.0"/>
             <parent link="base_footprint"/>
             <child link="base_link"/>
         </joint>
-        <!-- 给 gazebo 提供的标签【颜色...】 -->
         <gazebo reference="base_link">
             <material>Gazebo/Grey</material>

File: chapter6/chapt6_ws/install/robot_description2/share/robot_description2/urdf/robot/common_inertia.xacro (robot description, xacro)
@@ -1,6 +1,4 @@
 <?xml version="1.0"?>
 <robot xmlns:xacro="http://ros.org/wiki/xacro">
-    <!-- 长方体：{质量:. 长：， 宽：， 高：} -->
-    <!-- 单位：m千克 w、h、d米 -->
     <xacro:macro name="box_inertia" params="m w h d">
         <inertial>
@@ -9,5 +7,4 @@
         </inertial>
     </xacro:macro>
-    <!-- 圆柱体：{质量:. 半径：， 高度：} -->
     <xacro:macro name="cylinder_inertia" params="m r h">
         <inertial>
@@ -16,5 +13,4 @@
         </inertial>
     </xacro:macro>
-    <!-- 球体：{质量:. 半径：} -->
     <xacro:macro name="sphere_inertia" params="m r">
         <inertial>

File: chapter6/chapt6_ws/install/robot_description2/share/robot_description2/urdf/robot/plugins/gazebo_control_plugins.xacro (robot description, xacro)
@@ -3,36 +3,21 @@
     <xacro:macro name="gazebo_control_plugin">
         <gazebo>
-            <!-- <plugin name='插件的名字' filename='插件对应使用的文件【动态链接库】【/opt/ros/humble/lib/libgazebo_ros_diff_drive.so】'> -->
             <plugin name='diff_drive' filename='libgazebo_ros_diff_drive.so'>
-                <!-- 要传递给 ROS 的相关参数配置 -->
                 <ros>
-                    <!-- 所有话题前都加个“/”： “/cmd_vel” -->
                     <namespace>/</namespace>
                     <remapping>cmd_vel:=cmd_vel</remapping>
                     <remapping>odom:=odom</remapping>
                 </ros>
-                <!-- 发布消息的更新频率（单位：赫兹） -->
                 <update_rate>30</update_rate>
-                <!-- wheels：两轮差速模型 -->
                 <left_joint>left_wheel_joint</left_joint>
                 <right_joint>right_wheel_joint</right_joint>
-                <!-- kinematics -->
-                <!-- 轮距 -->
                 <wheel_separation>0.2</wheel_separation>
-                <!-- 轮子直径 -->
                 <wheel_diameter>0.064</wheel_diameter>
-                <!-- limits -->
-                <!-- 轮子的最大扭矩 -->
                 <max_wheel_torque>20</max_wheel_torque>
-                <!-- 轮子的最大加速度 -->
                 <max_wheel_acceleration>1.0</max_wheel_acceleration>
-                <!-- output：是否发布XXX -->
                 <publish_odom>true</publish_odom>
                 <publish_odom_tf>true</publish_odom_tf>
                 <publish_wheel_tf>true</publish_wheel_tf>
-                <!-- 坐标系名字 -->
-                <!-- 父坐标系 -->
                 <odometry_frame>odom</odometry_frame>
-                <!-- 子坐标系 -->
                 <robot_base_frame>base_footprint</robot_base_frame>
             </plugin>

File: chapter6/chapt6_ws/install/robot_description2/share/robot_description2/urdf/robot/plugins/gazebo_sensor_plugins.xacro (robot description, xacro)
@@ -16,34 +16,21 @@
                 <update_rate>5</update_rate>
                 <pose>0 0 0 0 0 0</pose>
-                <!-- 激光传感器配置 -->
                 <ray>
-                    <!-- 设置扫描范围 -->
                     <scan>
                         <horizontal>
-                            <!-- 水平上的采样点 -->
                             <samples>360</samples>
-                            <!-- 分辨率 -->
                             <resolution>1.000000</resolution>
-                            <!-- 最小角度【弧度制】 -->
                             <min_angle>0.000000</min_angle>
-                            <!-- 最大角度【弧度制】 -->
                             <max_angle>6.280000</max_angle>
                         </horizontal>
                     </scan>
-                    <!-- 设置扫描距离 -->
                     <range>
-                        <!-- 扫描距离【单位：米】 -->
                         <min>0.120000</min>
                         <max>8.0</max>
-                        <!-- 分辨率【雷达精度】 -->
                         <resolution>0.015000</resolution>
                     </range>
-                    <!-- 设置噪声【为了和真实的传感器更加相近】 -->
                     <noise>
-                        <!-- 高斯噪声 -->
                         <type>gaussian</type>
-                        <!-- 均值 -->
                         <mean>0.0</mean>
-                        <!-- 标准差 -->
                         <stddev>0.01</stddev>
                     </noise>
@@ -58,17 +45,11 @@
                         <remapping>~/out:=imu</remapping>
                     </ros>
-                    <!-- 不使用初始方向作为参考系 -->
                     <initial_orientation_as_reference>false</initial_orientation_as_reference>
                 </plugin>
-                <!-- 更新速率 -->
                 <update_rate>100</update_rate>
-                <!-- 传感器是否打开 -->
                 <always_on>true</always_on>
-                <!-- 六轴噪声设置 -->
                 <imu>
-                    <!-- 角速度 -->
                     <angular_velocity>
                         <x>
-                            <!-- 高斯噪声的设置 -->
                             <noise type="gaussian">
                                 <mean>0.0</mean>
@@ -95,5 +76,4 @@
                         </z>
                     </angular_velocity>
-                    <!-- 【线】加速度 -->
                     <linear_acceleration>
                         <x>

File: chapter6/chapt6_ws/install/robot_description2/share/robot_description2/urdf/robot/robot.urdf.xacro (robot description, xacro)
@@ -1,19 +1,13 @@
 <?xml version="1.0"?>
 <robot xmlns:xacro="http://www.ros.org/wiki/xacro" name="second_robot">
-<!-- 引入已经构建好的 xacro 文件 -->
-<!-- filename="$(find 功能包名字)/urdf/robot/xacro文件名" -->
-<!-- 基础部分 base_link -->
 <xacro:include filename="$(find robot_description2)/urdf/robot/base.urdf.xacro"/>
-<!-- 传感器部分 -->
 <xacro:include filename="$(find robot_description2)/urdf/robot/sensor/imu.urdf.xacro"/>
 <xacro:include filename="$(find robot_description2)/urdf/robot/sensor/camera.urdf.xacro"/>
 <xacro:include filename="$(find robot_description2)/urdf/robot/sensor/laser.urdf.xacro"/>
-<!-- 执行器部分 -->
 <xacro:include filename="$(find robot_description2)/urdf/robot/actuator/wheel.urdf.xacro"/>
 <xacro:include filename="$(find robot_description2)/urdf/robot/actuator/caster.urdf.xacro"/>
-<!-- 插件部分 -->
 <xacro:include filename="$(find robot_description2)/urdf/robot/plugins/gazebo_control_plugins.xacro"/>
 <xacro:include filename="$(find robot_description2)/urdf/robot/plugins/gazebo_sensor_plugins.xacro"/>
-<!-- 调用宏 xacro -->
+<xacro:include filename="$(find robot_description2)/urdf/robot/plugins/robot.ros2_control.xacro"/>
 <xacro:base_xacro length="0.12" radius="0.1"/>
 <xacro:imu_xacro xyz="0.0 0.0 0.02"/>
@@ -24,5 +18,5 @@
 <xacro:caster_xacro caster_name="front_caster" xyz="0.08 0.0 -0.076"/>
 <xacro:caster_xacro caster_name="back_caster" xyz="-0.08 0.0 -0.076"/>
-<xacro:gazebo_control_plugin/>
 <xacro:gazebo_sensor_plugin/>
+<xacro:robot_ros2_control/>
 </robot>

File: chapter6/chapt6_ws/install/robot_description2/share/robot_description2/urdf/robot/sensor/camera.urdf.xacro (robot description, xacro)
@@ -1,21 +1,13 @@
 <?xml version="1.0"?>
 <robot xmlns:xacro="http://www.ros.org/wiki/xacro">
-    <!-- 引入已经构建好的 xacro 文件 -->
     <xacro:include filename="$(find robot_description2)/urdf/robot/common_inertia.xacro"/>
     <xacro:macro name="camera_xacro" params="xyz">
-        <!-- 虚拟 link -->
         <link name="camera_optical_link"></link>
-        <!-- 机器人的 camera 部件 -->
         <link name="camera_link">
-            <!-- 部件的外观描述 -->
             <visual>
-                <!-- 沿着自己几何中心的偏移和旋转量 -->
                 <origin xyz="0.0 0.0 0.0" rpy="0.0 0.0 0.0"/>
-                <!-- 几何形状 -->
                 <geometry>
-                    <!-- 正方体：{长：， 宽：， 高：} -->
                     <box size="0.02 0.10 0.02"/>
                 </geometry>
-                <!-- 材质和颜色 -->
                 <material name="black">
                     <color rgba="0.0 0.0 0.0 0.5"/>
@@ -23,12 +15,8 @@
             </visual>
             <collision>
-                <!-- 沿着自己几何中心的偏移和旋转量 -->
                 <origin xyz="0.0 0.0 0.0" rpy="0.0 0.0 0.0"/>
-                <!-- 几何形状 -->
                 <geometry>
-                    <!-- 正方体：{长：， 宽：， 高：} -->
                     <box size="0.02 0.10 0.02"/>
                 </geometry>
-                <!-- 材质和颜色 -->
                 <material name="black">
                     <color rgba="0.0 0.0 0.0 0.5"/>
@@ -37,20 +25,14 @@
             <xacro:box_inertia m="0.1" w="0.02" h="0.10" d="0.02"/>
         </link>
-        <!-- 机器人的关节，用于组合机器人的部件 -->
         <joint name="camera_joint" type="fixed">
             <parent link="base_link"/>
             <child link="camera_link"/>
-            <!-- 将 camera 固定在 base_link 几何中心的偏移处 -->
             <origin xyz="${xyz}" rpy="0.0 0.0 0.0"/>
         </joint>
-        <!-- 机器人的关节，用于组合机器人的部件 -->
         <joint name="camera_optical_joint" type="fixed">
             <parent link="camera_link"/>
             <child link="camera_optical_link"/>
-            <!-- 将 camera_optical_link 固定在 camera_link 几何中心的偏移处 -->
-            <!-- 相机朝向默认前方为 z 轴，因此要进行修正，旋转 90 度 -->
             <origin xyz="0.0 0.0 0.0" rpy="${-pi/2} 0.0 ${-pi/2}"/>
         </joint>
-        <!-- 给 gazebo 提供的标签【颜色...】 -->
         <gazebo reference="camera_link">
             <material>Gazebo/Black</material>

File: chapter6/chapt6_ws/install/robot_description2/share/robot_description2/urdf/robot/sensor/imu.urdf.xacro (robot description, xacro)
@@ -1,19 +1,12 @@
 <?xml version="1.0"?>
 <robot xmlns:xacro="http://www.ros.org/wiki/xacro">
-    <!-- 引入已经构建好的 xacro 文件 -->
     <xacro:include filename="$(find robot_description2)/urdf/robot/common_inertia.xacro"/>
     <xacro:macro name="imu_xacro" params="xyz">
-        <!-- 机器人的 IMU 部件，惯性测量传感器 -->
         <link name="imu_link">
-            <!-- 部件的外观描述 -->
             <visual>
-                <!-- 沿着自己几何中心的偏移和旋转量 -->
                 <origin xyz="0.0 0.0 0.0" rpy="0.0 0.0 0.0"/>
-                <!-- 几何形状 -->
                 <geometry>
-                    <!-- 正方体：{长：， 宽：， 高：} -->
                     <box size="0.02 0.02 0.02"/>
                 </geometry>
-                <!-- 材质和颜色 -->
                 <material name="black">
                     <color rgba="0.0 0.0 0.0 0.5"/>
@@ -21,12 +14,8 @@
             </visual>
             <collision>
-                <!-- 沿着自己几何中心的偏移和旋转量 -->
                 <origin xyz="0.0 0.0 0.0" rpy="0.0 0.0 0.0"/>
-                <!-- 几何形状 -->
                 <geometry>
-                    <!-- 正方体：{长：， 宽：， 高：} -->
                     <box size="0.02 0.02 0.02"/>
                 </geometry>
-                <!-- 材质和颜色 -->
                 <material name="black">
                     <color rgba="0.0 0.0 0.0 0.5"/>
@@ -35,12 +24,9 @@
             <xacro:box_inertia m="0.05" w="0.02" h="0.02" d="0.02"/>
         </link>
-        <!-- 机器人的关节，用于组合机器人的部件 -->
         <joint name="imu_joint" type="fixed">
             <parent link="base_link"/>
             <child link="imu_link"/>
-            <!-- 将 imu 固定在 base_link 几何中心的偏移处 -->
             <origin xyz="${xyz}" rpy="0.0 0.0 0.0"/>
         </joint>
-        <!-- 给 gazebo 提供的标签【颜色...】 -->
         <gazebo reference="imu_link">
             <material>Gazebo/Red</material>

File: chapter6/chapt6_ws/install/robot_description2/share/robot_description2/urdf/robot/sensor/laser.urdf.xacro (robot description, xacro)
@@ -1,18 +1,12 @@
 <?xml version="1.0"?>
 <robot xmlns:xacro="http://www.ros.org/wiki/xacro">
-    <!-- 引入已经构建好的 xacro 文件 -->
     <xacro:include filename="$(find robot_description2)/urdf/robot/common_inertia.xacro"/>
     <xacro:macro name="laser_xacro" params="xyz">
-        <!-- 机器人的 laser 支撑杆部件 -->
         <link name="laser_cylinder_link">
-            <!-- 部件的外观描述 -->
             <visual>
-                <!-- 沿着自己几何中心的偏移和旋转量 -->
                 <origin xyz="0.0 0.0 0.0" rpy="0.0 0.0 0.0"/>
-                <!-- 几何形状 -->
                 <geometry>
                     <cylinder radius="0.01" length="0.10"/>
                 </geometry>
-                <!-- 材质和颜色 -->
                 <material name="black">
                     <color rgba="0.0 0.0 0.0 1.0"/>
@@ -20,11 +14,8 @@
             </visual>
             <collision>
-                <!-- 沿着自己几何中心的偏移和旋转量 -->
                 <origin xyz="0.0 0.0 0.0" rpy="0.0 0.0 0.0"/>
-                <!-- 几何形状 -->
                 <geometry>
                     <cylinder radius="0.01" length="0.10"/>
                 </geometry>
-                <!-- 材质和颜色 -->
                 <material name="black">
                     <color rgba="0.0 0.0 0.0 1.0"/>
@@ -33,15 +24,10 @@
             <xacro:cylinder_inertia m="0.05" r="0.01" h="0.10"/>
         </link>
-        <!-- 雷达部件 -->
         <link name="laser_link">
-            <!-- 部件的外观描述 -->
             <visual>
-                <!-- 沿着自己几何中心的偏移和旋转量 -->
                 <origin xyz="0.0 0.0 0.0" rpy="0.0 0.0 0.0"/>
-                <!-- 几何形状 -->
                 <geometry>
                     <cylinder radius="0.02" length="0.02"/>
                 </geometry>
-                <!-- 材质和颜色 -->
                 <material name="black">
                     <color rgba="0.0 0.0 0.0 1.0"/>
@@ -49,11 +35,8 @@
             </visual>
             <collision>
-                <!-- 沿着自己几何中心的偏移和旋转量 -->
                 <origin xyz="0.0 0.0 0.0" rpy="0.0 0.0 0.0"/>
-                <!-- 几何形状 -->
                 <geometry>
                     <cylinder radius="0.02" length="0.02"/>
                 </geometry>
-                <!-- 材质和颜色 -->
                 <material name="black">
                     <color rgba="0.0 0.0 0.0 1.0"/>
@@ -62,22 +45,14 @@
             <xacro:cylinder_inertia m="0.10" r="0.02" h="0.02"/>
         </link>
-        <!-- 机器人的关节，用于组合机器人的部件 -->
-        <!-- 将雷达固定到支撑杆上 -->
         <joint name="laser_joint" type="fixed">
             <parent link="laser_cylinder_link"/>
             <child link="laser_link"/>
-            <!-- 将 laser_link 固定在 laser_cylinder_link 几何中心的偏移处 -->
-            <!-- 因为雷达支撑杆的高度为 0.10米，因此几何中心处为 0.05米 -->
             <origin xyz="0.0 0.0 0.05" rpy="0.0 0.0 0.0"/>
         </joint>
-        <!-- 机器人的关节，用于组合机器人的部件 -->
-        <!-- 将雷达支撑杆固定到 base_link 上 -->
         <joint name="laser_cylinder_joint" type="fixed">
             <parent link="base_link"/>
             <child link="laser_cylinder_link"/>
-            <!-- 将 laser_cylinder_link 固定在 base_link 几何中心的偏移处 -->
             <origin xyz="${xyz}" rpy="0.0 0.0 0.0"/>
         </joint>
-        <!-- 给 gazebo 提供的标签【颜色...】 -->
         <gazebo reference="laser_cylinder_link">
             <material>Gazebo/Black</material>
