Commit message: code update

File: chapter6/chapt6_ws/src/robot_description2/urdf/robot/plugins/gazebo_sensor_plugins.xacro (robot description, xacro)
@@ -16,34 +16,21 @@
                 <update_rate>5</update_rate>
                 <pose>0 0 0 0 0 0</pose>
-                <!-- 激光传感器配置 -->
                 <ray>
-                    <!-- 设置扫描范围 -->
                     <scan>
                         <horizontal>
-                            <!-- 水平上的采样点 -->
                             <samples>360</samples>
-                            <!-- 分辨率 -->
                             <resolution>1.000000</resolution>
-                            <!-- 最小角度【弧度制】 -->
                             <min_angle>0.000000</min_angle>
-                            <!-- 最大角度【弧度制】 -->
                             <max_angle>6.280000</max_angle>
                         </horizontal>
                     </scan>
-                    <!-- 设置扫描距离 -->
                     <range>
-                        <!-- 扫描距离【单位：米】 -->
                         <min>0.120000</min>
                         <max>8.0</max>
-                        <!-- 分辨率【雷达精度】 -->
                         <resolution>0.015000</resolution>
                     </range>
-                    <!-- 设置噪声【为了和真实的传感器更加相近】 -->
                     <noise>
-                        <!-- 高斯噪声 -->
                         <type>gaussian</type>
-                        <!-- 均值 -->
                         <mean>0.0</mean>
-                        <!-- 标准差 -->
                         <stddev>0.01</stddev>
                     </noise>
@@ -58,17 +45,11 @@
                         <remapping>~/out:=imu</remapping>
                     </ros>
-                    <!-- 不使用初始方向作为参考系 -->
                     <initial_orientation_as_reference>false</initial_orientation_as_reference>
                 </plugin>
-                <!-- 更新速率 -->
                 <update_rate>100</update_rate>
-                <!-- 传感器是否打开 -->
                 <always_on>true</always_on>
-                <!-- 六轴噪声设置 -->
                 <imu>
-                    <!-- 角速度 -->
                     <angular_velocity>
                         <x>
-                            <!-- 高斯噪声的设置 -->
                             <noise type="gaussian">
                                 <mean>0.0</mean>
@@ -95,5 +76,4 @@
                         </z>
                     </angular_velocity>
-                    <!-- 【线】加速度 -->
                     <linear_acceleration>
                         <x>
@@ -130,12 +110,8 @@
                     <frame_name>camera_optical_link</frame_name>
                 </plugin>
-                <!-- 是否开启相机 -->
                 <always_on>true</always_on>
-                <!-- 更新速率 -->
                 <update_rate>10</update_rate>
                 <camera name="camera">
-                    <!-- 水平视角配置 -->
                     <horizontal_fov>1.5009831567</horizontal_fov>
-                    <!-- 图像的宽、高、图像类型【RGB】 -->
                     <image>
                         <width>800</width>
@@ -143,5 +119,4 @@
                         <format>R8G8B8</format>
                     </image>
-                    <!-- 畸变系数 -->
                     <distortion>
                         <k1>0.0</k1>
@@ -150,5 +125,4 @@
                         <p1>0.0</p1>
                         <p2>0.0</p2>
-                        <!-- 图像中心坐标【x, y】 -->
                         <center>0.5 0.5</center>
                     </distortion>
