Commit message: code update

File: chapter6/chapt6_ws/install/robot_description2/share/robot_description2/urdf/robot/actuator/wheel.urdf.xacro (robot description, xacro)
@@ -28,4 +28,5 @@
             <child link="${wheel_name}_link"/>
             <origin xyz="${xyz}" rpy="0.0 0.0 0.0"/>
+            <axis xyz="0.0 1.0 0.0"/>
         </joint>
         <gazebo reference="${wheel_name}_link">
